File: hardware/dryer-mains/dryer-mains.kicad_pcb (KiCad board)
At the start: 2 copper layers, 45 x 70 mm, 19 parts, among them K1 SRD-05VDC-SL-C, K2 SRD-05VDC-SL-C, Q1 MMBT2222A, Q2 MMBT2222A

Commit message: Make the mains plug vertical and the fuse holder 12.5 mm after the second review
JWardT3D (PR #49, 2026-10-15): a wall borders the mains space, so the
plug's wires must leave perpendicular to the board; the fuse holders on
hand measure about 12.5 mm pitch with a 25.7 x 10 mm body.

J_MAINS becomes the vertical DORABO DB2EV-5.08-8P-GN (LCSC C395787) on a
local copy of the Phoenix MSTBVA 8-pin footprint drilled 1.7 mm, placed
at (39.5, 17.94) rotated 270 so pin 1 is the top pin and the body's
deeper side faces the edge; the housing no longer overhangs the board,
and test_outlines no longer allows any overhang. The DB2EV's own drawing
is not retrieved: the entry direction, the hole size and the body
envelope are inferred from the DB2EVC/DB2ERC drawings and the MSTBVA
footprint, and the docs say so. F1 moves to (15.6, 14) on a new 12.5 mm
slotted footprint (slots take 11.5 to 13.5 mm, body drawn centred on the
pins); the body fills the 26.2 mm between the slot and the plug's
courtyard with the two courtyards 0.16 mm apart. The 22.5 mm footprint
stays in the library because the measured pitch conflicts with the
BLX-A drawing that body matches (22.3 +-1.0): the docs and the
continuity checklist ask for the pin positions to be confirmed before
ordering.

The mains copper is re-laid: L_FUSED takes the x 21 spine on F.Cu from
F1's pad 2 to both COM pads with a branch at y 49.6 to pin 7; L_IN runs
from pad 1 over the top of the fuse body at y 9.6 and drops to pin 1;
L_SW_A goes straight from K1's NO pad to pin 3 and L_SW_B up the x 30.5
lane on B.Cu to pin 5, no longer crossing; the N links stay at x 43.15.
The SELV routing is unchanged and still DRC-clean against the new
copper, so the board is regenerated, not re-routed. Measured: 6.285 mm
mains to SELV outside the relay areas (F1 pad 1 to K1's coil pad),
1.850 mm between L-side nets (the pin-7 branch to K2's NC pad), 1.050 mm
to the edge, 7.536 mm to the nearest hole; the saved fill is 15.26 mm
from mains copper outside th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
Parts:
- removed the J_MAINS at (39.5, 53.5)
- added J_MAINS: 120 VAC, dryer:PhoenixContact_MSTBVA_2,5_8-G-5,08_1x08_P5.08mm_Vertical_Drill1.7mm, F.Cu at (39.5, 17.9)
- F1: footprint dryer:Fuseholder_5x20mm_Covered_P22.50mm_Slot -> dryer:Fuseholder_5x20mm_Covered_P12.50mm_Slot
- moved F1 3.20 mm to (15.6, 14.0)
Routing:
- net L_IN: track 64.8 -> 32.0 mm
- net L_SW_B: track 35.2 -> 30.1 mm
- net L_SW_A: track 16.8 -> 15.1 mm
- net L_FUSED: track 81.3 -> 79.8 mm

Commit message: Fit the fab-fitted 15 mm fuse holder after the reviewer confirmed the on-hand pitch
JWardT3D (PR #49, 2026-10-15): the holders on hand are about 22 mm
pitch after all (the 12.5 mm came from the listing's picture); the hole
pattern, the USB-C overhang, the vertical plug and the strip-to-COM
clearance stand; the plug's screws should face away from the wall.

Their 25.8 mm BLX-A body and the vertical plug do not both fit: with
mains copper 1 mm from the slot the body runs from x 10.35 to 36.15,
0.56 mm into the plug's body and 1 mm into its courtyard at 35.16
(strip, slot, clearance, holder and plug body add up to 45.6 mm across
the 45 mm board). F1 therefore returns to the single-board rev A's
XFCN PTF-76-B (LCSC C48603682, 15 mm pitch, UL 250 VAC 20 A),
fab-fitted, at (28.7, 14) rotated 180 so its L_IN pad is on the plug
side, one short diagonal from pin 1, and its L_FUSED pad feeds the
spine; the body sits flush with the slot edge, 1.5 mm short of the
plug's courtyard. The 12.5 mm footprint is removed; the 22.5 mm slotted
one stays in the library for a right-angle-plug layout, where the
holders on hand fit. The L_IN run over the fuse body is gone. Which
side the plug's screws face is recorded as unverified (the DB2EV
drawing is not on file); turning the header 180 is the fix if needed.

The strip's driver A is back where it was; the SELV nets are re-routed
(119 tracks and 12 vias). Measured: 6.303 mm mains to SELV outside the
relay areas (F1 pad 2 to K1's coil pad), 1.850 mm between L-side nets,
1.050 mm to the edge, 9.229 mm to the nearest hole, SELV copper 3.950 mm
from a COM pad (strip 4.407; the reviewer accepted 4.05 before the
re-route), saved fill 4.000 mm inside the areas and 10.17 outside. No
part is hand-fitted on the mains board now; the tests, BOM table,
continuity checklist, both specs, the datasheet index, CLAUDE.md and
the README follow.

Co-Authored-By: Claude Fable 5.1 <noreply@anthropic.com>
Parts:
- F1: footprint dryer:Fuseholder_5x20mm_Covered_P12.50mm_Slot -> dryer:Fuseholder_5x20mm_Covered_XFCN_PTF-76-B_P15.00mm
- moved F1 13.1 mm to (28.7, 14.0), turned to 180 degrees
Routing:
- net L_IN: track 32.0 -> 11.5 mm
- net +5V: track 91.7 -> 77.5 mm, vias 3 -> 4
- net RLY_A: track 31.1 -> 22.5 mm, vias 4 -> 0
- net GND: track 37.8 -> 40.1 mm, vias 2 -> 3
- net COIL_A: track 39.4 -> 37.2 mm
