File: hardware/dryer-mains/dryer-mains.kicad_sch (KiCad schematic)
At the start: 19 parts, among them K1 SRD-05VDC-SL-C, K2 SRD-05VDC-SL-C, Q1 MMBT2222A, Q2 MMBT2222A

Commit message: Make the mains plug vertical and the fuse holder 12.5 mm after the second review
JWardT3D (PR #49, 2026-10-15): a wall borders the mains space, so the
plug's wires must leave perpendicular to the board; the fuse holders on
hand measure about 12.5 mm pitch with a 25.7 x 10 mm body.

J_MAINS becomes the vertical DORABO DB2EV-5.08-8P-GN (LCSC C395787) on a
local copy of the Phoenix MSTBVA 8-pin footprint drilled 1.7 mm, placed
at (39.5, 17.94) rotated 270 so pin 1 is the top pin and the body's
deeper side faces the edge; the housing no longer overhangs the board,
and test_outlines no longer allows any overhang. The DB2EV's own drawing
is not retrieved: the entry direction, the hole size and the body
envelope are inferred from the DB2EVC/DB2ERC drawings and the MSTBVA
footprint, and the docs say so. F1 moves to (15.6, 14) on a new 12.5 mm
slotted footprint (slots take 11.5 to 13.5 mm, body drawn centred on the
pins); the body fills the 26.2 mm between the slot and the plug's
courtyard with the two courtyards 0.16 mm apart. The 22.5 mm footprint
stays in the library because the measured pitch conflicts with the
BLX-A drawing that body matches (22.3 +-1.0): the docs and the
continuity checklist ask for the pin positions to be confirmed before
ordering.

The mains copper is re-laid: L_FUSED takes the x 21 spine on F.Cu from
F1's pad 2 to both COM pads with a branch at y 49.6 to pin 7; L_IN runs
from pad 1 over the top of the fuse body at y 9.6 and drops to pin 1;
L_SW_A goes straight from K1's NO pad to pin 3 and L_SW_B up the x 30.5
lane on B.Cu to pin 5, no longer crossing; the N links stay at x 43.15.
The SELV routing is unchanged and still DRC-clean against the new
copper, so the board is regenerated, not re-routed. Measured: 6.285 mm
mains to SELV outside the relay areas (F1 pad 1 to K1's coil pad),
1.850 mm between L-side nets (the pin-7 branch to K2's NC pad), 1.050 mm
to the edge, 7.536 mm to the nearest hole; the saved fill is 15.26 mm
from mains copper outside th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
Parts:
- F1: footprint dryer:Fuseholder_5x20mm_Covered_P22.50mm_Slot -> dryer:Fuseholder_5x20mm_Covered_P12.50mm_Slot
- J_MAINS: footprint dryer:PhoenixContact_MSTBA_2,5_8-G-5,08_1x08_P5.08mm_Horizontal_Drill1.7mm -> dryer:PhoenixContact_MSTBVA_2,5_8-G-5,08_1x08_P5.08mm_Vertical_Drill1.7mm; LCSC C395786 -> C395787
Changed lines of the file:
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@@
 (no_connect (at 104.14 55.88))
 (global_label "COIL_B" (shape input) (at 96.52 55.88 90) (effects (font (size 1.27 1.27)) (justify left)))
-(symbol (lib_id "Device:Fuse") (at 139.70 63.50 0) (unit 1) (exclude_from_sim no) (in_bom yes) (on_board yes) (dnp no) (property "Reference" "F1" (at 139.70 60.96 0) (effects (font (size 1.27 1.27)))) (property "Value" "T 3.15 A 5x20" (at 139.70 66.04 0) (effects (font (size 1.27 1.27)))) (property "Footprint" "dryer:Fuseholder_5x20mm_Covered_P22.50mm_Slot" (at 139.70 63.50 0) (effects (font (size 1.27 1.27)) (hide yes))) (property "Datasheet" "~" (at 139.70 63.50 0) (effects (font (size 1.27 1.27)) (hide yes))) (property "LCSC" "" (at 139.70 63.50 0) (effects (font (size 1.27 1.27)) (hide yes))) (property "Description" "covered 5 x 20 mm holder on 22.5 mm pitch, slotted holes for 21.5 to 23.5 mm: hand-fitted from the BLX-A style holders on hand (Amazon B0FCS5MK1Y, 10 A 250 V, pitch 22.3 +-1.0 mm by the moulding's datasheet, not stated by the seller: measure one, hardware/README.md); the fab-fitted alternative is XFCN PTF-77 C717030 (22.50 mm, UL 250 VAC 20 A, same body as the PTF-76-B), JLCPCB extended. The T 3.15 A fuse itself is fitted by hand" (at 139.70 63.50 0) (effects (font (size 1.27 1.27)) (hide yes))) (property "Hand fit" "yes" (at 139.70 63.50 0) (effects (font (size 1.27 1.27)) (hide yes))) (pin "1") (pin "2") (instances (project "dryer-mains" (path "/97ff8b13-3eed-5268-af54-f6b8bdb155b7" (reference "F1") (unit 1)))))
+(symbol (lib_id "Device:Fuse") (at 139.70 63.50 0) (unit 1) (exclude_from_sim no) (in_bom yes) (on_board yes) (dnp no) (property "Reference" "F1" (at 139.70 60.96 0) (effects (font (size 1.27 1.27)))) (property "Value" "T 3.15 A 5x20" (at 139.70 66.04 0) (effects (font (size 1.27 1.27)))) (property "Footprint" "dryer:Fuseholder_5x20mm_Covered_P12.50mm_Slot" (at 139.70 63.50 0) (effects (font (size 1.27 1.27)) (hide yes))) (property "Datasheet" "~" (at 139.70 63.50 0) (effects (font (size 1.27 1.27)) (hide yes))) (property "LCSC" "" (at 139.70 63.50 0) (effects (font (size 1.27 1.27)) (hide yes))) (property "Description" "covered 5 x 20 mm holder, hand-fitted from the holders on hand (Amazon B0FCS5MK1Y, 10 A 250 V), drawn to the hardware reviewer's measurement of 2026-10-15: pins about 12.5 mm apart, body 25.7 x 10 mm; slotted holes take 11.5 to 13.5 mm. That pitch conflicts with the BLX-A drawing the body matches (22.3 +-1.0 mm), so confirm the pin positions before ordering; the 22.5 mm slotted footprint stays in hardware/lib/dryer.pretty (hardware/README.md). The T 3.15 A fuse itself is fitted by hand" (at 139.70 63.50 0) (effects (font (size 1.27 1.27)) (hide yes))) (property "Hand fit" "yes" (at 139.70 63.50 0) (effects (font (size 1.27 1.27)) (hide yes))) (pin "1") (pin "2") (instances (project "dryer-mains" (path "/97ff8b13-3eed-5268-af54-f6b8bdb155b7" (reference "F1") (unit 1)))))
 (global_label "L_IN" (shape input) (at 139.70 59.69 90) (effects (font (size 1.27 1.27)) (justify left)))
 (global_label "L_FUSED" (shape input) (at 139.70 67.31 270) (effects (font (size 1.27 1.27)) (justify left)))
-(symbol (lib_id "Connector_Generic:Conn_01x08") (at 177.80 63.50 0) (unit 1) (exclude_from_sim no) (in_bom yes) (on_board yes) (dnp no) (property "Reference" "J_MAINS" (at 177.80 60.96 0) (effects (font (size 1.27 1.27)))) (property "Value" "120 VAC" (at 177.80 66.04 0) (effects (font (size 1.27 1.27)))) (property "Footprint" "dryer:PhoenixContact_MSTBA_2,5_8-G-5,08_1x08_P5.08mm_Horizontal_Drill1.7mm" (at 177.80 63.50 0) (effects (font (size 1.27 1.27)) (hide yes))) (property "Datasheet" "~" (at 177.80 63.50 0) (effects (font (size 1.27 1.27)) (hide yes))) (property "LCSC" "C395786" (at 177.80 63.50 0) (effects (font (size 1.27 1.27)) (hide yes))) (property "Description" "L in, N in, heater A L-sw/N, heater B L-sw/N, PSU L (fused)/N; DORABO DB2ERC-5.08-8P-GN, right angle, 300 V 15 A (UL); plug DB2EK-5.08-8P-GN-S C395791, loose; JLCPCB extended" (at 177.80 63.50 0) (effects (font (size 1.27 1.27)) (hide yes))) (pin "1") (pin "2") (pin "3") (pin "4") (pin "5") (pin "6") (pin "7") (pin "8") (instances (project "dryer-mains" (path "/97ff8b13-3eed-5268-af54-f6b8bdb155b7" (reference "J_MAINS") (unit 1)))))
+(symbol (lib_id "Connector_Generic:Conn_01x08") (at 177.80 63.50 0) (unit 1) (exclude_from_sim no) (in_bom yes) (on_board yes) (dnp no) (property "Reference" "J_MAINS" (at 177.80 60.96 0) (effects (font (size 1.27 1.27)))) (property "Value" "120 VAC" (at 177.80 66.04 0) (effects (font (size 1.27 1.27)))) (property "Footprint" "dryer:PhoenixContact_MSTBVA_2,5_8-G-5,08_1x08_P5.08mm_Vertical_Drill1.7mm" (at 177.80 63.50 0) (effects (font (size 1.27 1.27)) (hide yes))) (property "Datasheet" "~" (at 177.80 63.50 0) (effects (font (size 1.27 1.27)) (hide yes))) (property "LCSC" "C395787" (at 177.80 63.50 0) (effects (font (size 1.27 1.27)) (hide yes))) (property "Description" "L in, N in, heater A L-sw/N, heater B L-sw/N, PSU L (fused)/N; DORABO DB2EV-5.08-8P-GN, vertical (wires perpendicular to the board: a wall borders the mains space, reviewer 2026-10-15), 630 V 15 A per LCSC. Its drawing is not retrieved: the vertical entry is inferred from the series letter and LCSC's open-side listing, the 1.7 mm holes and the body from the DB2EVC/DB2ERC drawings and the MSTBVA footprint; confirm before ordering. Plug DB2EK-5.08-8P-GN-S C395791, loose; JLCPCB extended" (at 177.80 63.50 0) (effects (font (size 1.27 1.27)) (hide yes))) (pin "1") (pin "2") (pin "3") (pin "4") (pin "5") (pin "6") (pin "7") (pin "8") (instances (project "dryer-mains" (path "/97ff8b13-3eed-5268-af54-f6b8bdb155b7" (reference "J_MAINS") (unit 1)))))
 (global_label "L_IN" (shape input) (at 172.72 55.88 180) (effects (font (size 1.27 1.27)) (justify left)))
 (global_label "N" (shape input) (at 172.72 58.42 180) (effects (font (size 1.27 1.27)) (justify left)))

Commit message: Fit the fab-fitted 15 mm fuse holder after the reviewer confirmed the on-hand pitch
JWardT3D (PR #49, 2026-10-15): the holders on hand are about 22 mm
pitch after all (the 12.5 mm came from the listing's picture); the hole
pattern, the USB-C overhang, the vertical plug and the strip-to-COM
clearance stand; the plug's screws should face away from the wall.

Their 25.8 mm BLX-A body and the vertical plug do not both fit: with
mains copper 1 mm from the slot the body runs from x 10.35 to 36.15,
0.56 mm into the plug's body and 1 mm into its courtyard at 35.16
(strip, slot, clearance, holder and plug body add up to 45.6 mm across
the 45 mm board). F1 therefore returns to the single-board rev A's
XFCN PTF-76-B (LCSC C48603682, 15 mm pitch, UL 250 VAC 20 A),
fab-fitted, at (28.7, 14) rotated 180 so its L_IN pad is on the plug
side, one short diagonal from pin 1, and its L_FUSED pad feeds the
spine; the body sits flush with the slot edge, 1.5 mm short of the
plug's courtyard. The 12.5 mm footprint is removed; the 22.5 mm slotted
one stays in the library for a right-angle-plug layout, where the
holders on hand fit. The L_IN run over the fuse body is gone. Which
side the plug's screws face is recorded as unverified (the DB2EV
drawing is not on file); turning the header 180 is the fix if needed.

The strip's driver A is back where it was; the SELV nets are re-routed
(119 tracks and 12 vias). Measured: 6.303 mm mains to SELV outside the
relay areas (F1 pad 2 to K1's coil pad), 1.850 mm between L-side nets,
1.050 mm to the edge, 9.229 mm to the nearest hole, SELV copper 3.950 mm
from a COM pad (strip 4.407; the reviewer accepted 4.05 before the
re-route), saved fill 4.000 mm inside the areas and 10.17 outside. No
part is hand-fitted on the mains board now; the tests, BOM table,
continuity checklist, both specs, the datasheet index, CLAUDE.md and
the README follow.

Co-Authored-By: Claude Fable 5.1 <noreply@anthropic.com>
Parts:
- F1: footprint dryer:Fuseholder_5x20mm_Covered_P12.50mm_Slot -> dryer:Fuseholder_5x20mm_Covered_XFCN_PTF-76-B_P15.00mm; Hand fit yes -> (none); LCSC (none) -> C48603682
Changed lines of the file:
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@@
 (no_connect (at 104.14 55.88))
 (global_label "COIL_B" (shape input) (at 96.52 55.88 90) (effects (font (size 1.27 1.27)) (justify left)))
-(symbol (lib_id "Device:Fuse") (at 139.70 63.50 0) (unit 1) (exclude_from_sim no) (in_bom yes) (on_board yes) (dnp no) (property "Reference" "F1" (at 139.70 60.96 0) (effects (font (size 1.27 1.27)))) (property "Value" "T 3.15 A 5x20" (at 139.70 66.04 0) (effects (font (size 1.27 1.27)))) (property "Footprint" "dryer:Fuseholder_5x20mm_Covered_P12.50mm_Slot" (at 139.70 63.50 0) (effects (font (size 1.27 1.27)) (hide yes))) (property "Datasheet" "~" (at 139.70 63.50 0) (effects (font (size 1.27 1.27)) (hide yes))) (property "LCSC" "" (at 139.70 63.50 0) (effects (font (size 1.27 1.27)) (hide yes))) (property "Description" "covered 5 x 20 mm holder, hand-fitted from the holders on hand (Amazon B0FCS5MK1Y, 10 A 250 V), drawn to the hardware reviewer's measurement of 2026-10-15: pins about 12.5 mm apart, body 25.7 x 10 mm; slotted holes take 11.5 to 13.5 mm. That pitch conflicts with the BLX-A drawing the body matches (22.3 +-1.0 mm), so confirm the pin positions before ordering; the 22.5 mm slotted footprint stays in hardware/lib/dryer.pretty (hardware/README.md). The T 3.15 A fuse itself is fitted by hand" (at 139.70 63.50 0) (effects (font (size 1.27 1.27)) (hide yes))) (property "Hand fit" "yes" (at 139.70 63.50 0) (effects (font (size 1.27 1.27)) (hide yes))) (pin "1") (pin "2") (instances (project "dryer-mains" (path "/97ff8b13-3eed-5268-af54-f6b8bdb155b7" (reference "F1") (unit 1)))))
+(symbol (lib_id "Device:Fuse") (at 139.70 63.50 0) (unit 1) (exclude_from_sim no) (in_bom yes) (on_board yes) (dnp no) (property "Reference" "F1" (at 139.70 60.96 0) (effects (font (size 1.27 1.27)))) (property "Value" "T 3.15 A 5x20" (at 139.70 66.04 0) (effects (font (size 1.27 1.27)))) (property "Footprint" "dryer:Fuseholder_5x20mm_Covered_XFCN_PTF-76-B_P15.00mm" (at 139.70 63.50 0) (effects (font (size 1.27 1.27)) (hide yes))) (property "Datasheet" "~" (at 139.70 63.50 0) (effects (font (size 1.27 1.27)) (hide yes))) (property "LCSC" "C48603682" (at 139.70 63.50 0) (effects (font (size 1.27 1.27)) (hide yes))) (property "Description" "XFCN PTF-76-B covered 5 x 20 mm holder with lift-off cap, 15 mm pitch, UL 250 VAC 20 A, rev A's original choice, fab-fitted, JLCPCB extended. Chosen again on 2026-10-15: the BLX-A holders on hand (25.8 mm body, about 22 mm pitch as the reviewer confirmed, 22.3 on the drawing) and the vertical mains plug do not both fit across the 45 mm board once mains copper keeps 1 mm from the slot (the sum is 45.6 mm); the 22.5 mm slotted footprint stays in hardware/lib/dryer.pretty for a right-angle-plug layout. The T 3.15 A fuse itself is fitted by hand" (at 139.70 63.50 0) (effects (font (size 1.27 1.27)) (hide yes))) (pin "1") (pin "2") (instances (project "dryer-mains" (path "/97ff8b13-3eed-5268-af54-f6b8bdb155b7" (reference "F1") (unit 1)))))
 (global_label "L_IN" (shape input) (at 139.70 59.69 90) (effects (font (size 1.27 1.27)) (justify left)))
 (global_label "L_FUSED" (shape input) (at 139.70 67.31 270) (effects (font (size 1.27 1.27)) (justify left)))
